File: 2025/mathpad/mathpad.kicad_pcb (KiCad board)
At the start: 2 copper layers, 89 parts, among them J1 SWD, J2 Conn_01x31_Shielded, P1 USB_C_Plug_USB2.0, SW1 SW_Push, SW10 SW_Push, SW11 SW_Push, SW12 SW_Push, SW13 SW_Push, SW14 SW_Push, SW15 SW_Push, SW16 SW_Push, SW17 SW_Push, SW18 SW_Push, SW19 SW_Push, SW2 SW_Push, SW20 SW_Push, SW21 SW_Push, SW22 SW_Push, SW23 SW_Push, SW24 SW_Push, SW25 SW_Push, SW26 SW_Push, SW27 SW_Push, SW28 SW_Push, SW29 SW_Push, SW3 SW_Push, SW4 SW_Push, SW5 SW_Push, SW6 SW_Push, SW7 SW_Push, SW8 SW_Push, SW9 SW_Push, U1 STM32G0B1RCTx, U2 RT9078-33GJS, U3 TLV61046ADB, U4 RT9078-33GJS, Y1 Crystal_GND3_Small

Commit message: 20250422-1
Parts:
- added H1: MountingHole_Pad, MountingHole:MountingHole_2.2mm_M2_Pad, F.Cu at (54.0, 34.0)
- added H2: MountingHole_Pad, MountingHole:MountingHole_2.2mm_M2_Pad, F.Cu at (54.0, 181.0)
- added H3: MountingHole_Pad, MountingHole:MountingHole_2.2mm_M2_Pad, F.Cu at (141.0, 181.0)
- added H4: MountingHole_Pad, MountingHole:MountingHole_2.2mm_M2_Pad, F.Cu at (141.0, 34.0)
- C11: footprint Capacitor_SMD:C_0603_1608Metric -> Capacitor_SMD:C_1206_3216Metric
- moved D12 221.3 mm to (84.9, 175.9), turned to 180 degrees
- moved D6 220.4 mm to (65.9, 175.9), turned to 180 degrees
- moved D5 212.8 mm to (65.9, 156.9), turned to 180 degrees
- moved D11 212.7 mm to (84.9, 156.9), turned to 180 degrees
- moved D4 206.1 mm to (65.9, 137.8), turned to 180 degrees
- moved D3 200.3 mm to (65.9, 118.8), turned to 180 degrees
- moved C8 199.3 mm to (66.1, 37.5), turned to -90 degrees
- moved C10 198.7 mm to (83.0, 38.4), turned to -90 degrees
- moved C9 196.3 mm to (68.7, 37.5), turned to -90 degrees
- moved D2 195.6 mm to (65.9, 99.7), turned to 180 degrees
- moved D18 193.6 mm to (104.0, 175.9), turned to 180 degrees
- moved R3 192.2 mm to (78.3, 37.7), turned to -90 degrees
- moved R4 191.9 mm to (78.3, 41.1), turned to -90 degrees
- moved D23 191.6 mm to (123.0, 166.4), turned to 180 degrees
- moved D17 185.4 mm to (104.0, 156.9), turned to 180 degrees
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Connections:
- net Net-(U1-PA11/PA9) renamed /USB_N
- net Net-(U1-PA12/PA10) renamed /USB_P
- net USB_N renamed USB_CN_N
- net USB_P renamed USB_CN_P
Routing:
- net KEY_R6: track 0.00 -> 206.8 mm
- net KEY_R5: track 0.00 -> 195.1 mm
- net KEY_R4: track 0.00 -> 170.4 mm
- net KEY_R3: track 0.00 -> 152.2 mm
- net KEY_C5: track 0.00 -> 139.9 mm, vias 0 -> 1
- net KEY_C1: track 0.00 -> 139.7 mm, vias 0 -> 1
- net KEY_R2: track 0.00 -> 139.5 mm
- net KEY_C2: track 0.00 -> 122.3 mm, vias 0 -> 1
- net KEY_R1: track 0.00 -> 118.6 mm
- net KEY_C4: track 0.00 -> 113.1 mm, vias 0 -> 1
- net KEY_C3: track 0.00 -> 107.0 mm, vias 0 -> 1
- net VBUS: track 0.00 -> 52.9 mm, vias 0 -> 3
- net GND: track 0.00 -> 36.6 mm, vias 0 -> 19
- net USB_CN_P: track 0.00 -> 32.6 mm, vias 0 -> 2
- net USB_CN_N: track 0.00 -> 32.5 mm, vias 0 -> 2
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Other:
- board outline added: 95.2 x 155 mm
- copper layers 2 -> 4
- board text added: "MathPad {dblquote}Fort Myers{dblquote} Rev.B 20250421 CTCL 2022-2025"

Commit message: 20250423-1
Parts:
- L1: value L_Small -> 10uH
Routing:
- net VBUS: track 52.9 -> 135.8 mm, vias 3 -> 5
- net GND: track 36.6 -> 48.8 mm, vias 19 -> 76
- net (no net): vias 2 -> 0
- added copper zone on B.Cu, net GND
- added copper zone on F.Cu, net GND
Other:
- board text added: "MathPad {dblquote}Fort Myers{dblquote} Rev.B 20250422 CTCL 2022-2025"
- board text removed: "MathPad {dblquote}Fort Myers{dblquote} Rev.B 20250421 CTCL 2022-2025"
