File: 2025/mathpad/mathpad.kicad_sch (KiCad schematic)
At the start: 89 parts, among them J1 SWD, J2 Conn_01x31_Shielded, P1 USB_C_Plug_USB2.0, SW1 SW_Push, SW10 SW_Push, SW11 SW_Push, SW12 SW_Push, SW13 SW_Push, SW14 SW_Push, SW15 SW_Push, SW16 SW_Push, SW17 SW_Push, SW18 SW_Push, SW19 SW_Push, SW2 SW_Push, SW20 SW_Push, SW21 SW_Push, SW22 SW_Push, SW23 SW_Push, SW24 SW_Push, SW25 SW_Push, SW26 SW_Push, SW27 SW_Push, SW28 SW_Push, SW29 SW_Push, SW3 SW_Push, SW4 SW_Push, SW5 SW_Push, SW6 SW_Push, SW7 SW_Push, SW8 SW_Push, SW9 SW_Push, U1 STM32G0B1RCTx, U2 RT9078-33GJS, U3 TLV61046ADB, U4 RT9078-33GJS, Y1 Crystal_GND3_Small

Commit message: 20250422-1
Parts:
- added H1, H2, H3, H4: MountingHole_Pad, MountingHole:MountingHole_2.2mm_M2_Pad, symbol Mechanical:MountingHole_Pad
- C11: footprint Capacitor_SMD:C_0603_1608Metric -> Capacitor_SMD:C_1206_3216Metric
Connections:
- net USB_N: now also R1.1, U1.43 (PA11/PA9); no longer P1.A7 (D-), R1.2
- net USB_P: now also R2.1, U1.44 (PA12/PA10); no longer P1.A6 (D+), R2.2
- new net USB_CN_N: P1.A7 (D-), R1.2
- new net USB_CN_P: P1.A6 (D+), R2.2
Other:
- moved on the sheet: R1, R2

Commit message: 20250423-1
Parts:
- L1: value L_Small -> 10uH
Other:
- note added: "2025-04-18 - 2025-04-22"
- note added: "B"
- note added: "MathPad "Fort Myers""
- moved on the sheet: C10, C11, C12, C13, C14, C15, C16, C8, C9, D1, D10, D11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
